File: kicad/usbwledc-mosfet.kicad_pcb (KiCad board)
At the start: 4 copper layers, 40 x 35 mm, 37 parts, among them J1 5V OUT PAD, J10 USB_C_Receptacle_USB2.0, J2 D1 PAD, J3 GND PAD, J4 5V OUT PAD, J5 D2 PAD, J6 GND PAD, J7 Conn_01x04_Pin, Q1 IRLML6244, Q2 IRF7410TRPBF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

Commit message: Corrected JLC-Text
Other:
- board text added: "JLCJLCJLCJLV"
- board text removed: "JLCJLCJLC"
Changed lines of the file:
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@@
     (effects (font (size 1.5 1.5) (thickness 0.3) bold) (justify left bottom mirror))
   )
-  (gr_text "JLCJLCJLC" (at 29.5148 33.555356 90) (layer "B.SilkS")
+  (gr_text "JLCJLCJLCJLV" (at 29.5148 32.34107 90) (layer "B.SilkS")
     (effects (font (size 1 1) (thickness 0.15)) (justify left bottom mirror))
   )

Commit message: Corrected JLC-Text
Other:
- board text added: "JLCJLCJLCJLC"
- board text removed: "JLCJLCJLCJLV"
Changed lines of the file:
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@@
     (effects (font (size 1.5 1.5) (thickness 0.3) bold) (justify left bottom mirror))
   )
-  (gr_text "JLCJLCJLCJLV" (at 29.5148 32.34107 90) (layer "B.SilkS")
+  (gr_text "JLCJLCJLCJLC" (at 29.5148 32.34107 90) (layer "B.SilkS")
     (effects (font (size 1 1) (thickness 0.15)) (justify left bottom mirror))
   )
